File: hardware/kicad/KinderLight.kicad_sch (KiCad schematic)
At the start: 16 parts, among them J2 +5VCC, J3 ESP32C6 Left, J4 ESP32C6 Right, J5 5-24VCC, J7 I2C BH1750, J8 LED PWM, J9 +12VCC, Q1 AO3400A, Q2 AO3400A, Q3 AO3400A

Commit message: Added version 20260207 of the PCB
Parts:
- removed J2: +5VCC, Connector_PinHeader_2.00mm:PinHeader_1x08_P2.00mm_Vertical, symbol Connector_Generic:Conn_01x08
- removed J5: 5-24VCC, Connector_PinHeader_2.00mm:PinHeader_1x08_P2.00mm_Vertical, symbol Connector_Generic:Conn_01x08
- added H1, H2: MountingHole, MountingHole:MountingHole_3.2mm_M3, symbol Mechanical:MountingHole
- added J1: +5VCC, Connector_PinSocket_2.54mm:PinSocket_1x02_P2.54mm_Vertical, symbol Connector_Generic:Conn_01x02
- added J10: LED PWM JST, Connector_JST:JST_PH_B4B-PH-K_1x04_P2.00mm_Vertical, symbol Connector_Generic:Conn_01x04
- added J11: I2C BH1750 JST, Connector_JST:JST_PH_B4B-PH-K_1x04_P2.00mm_Vertical, symbol Connector_Generic:Conn_01x04
- added J2, J6: GND, Connector_PinSocket_2.54mm:PinSocket_1x02_P2.54mm_Vertical, symbol Connector_Generic:Conn_01x02
- added J5: VCC, Connector_PinSocket_2.54mm:PinSocket_1x02_P2.54mm_Vertical, symbol Connector_Generic:Conn_01x02
- J7, J8: LCSC (none) -> C161871
- J9: LCSC (none) -> C22397914
Connections:
- net GND: now also J11.2 (Pin_2), J2.1 (Pin_1), J2.2 (Pin_2), J6.1 (Pin_1), J6.2 (Pin_2)
- net I2C SCL: now also J11.3 (Pin_3)
- net I2C SDA: now also J11.4 (Pin_4)
- net VCC 12V MAX: now also J5.1 (Pin_1), J5.2 (Pin_2)
- net VCC 5V: now also J1.1 (Pin_1), J1.2 (Pin_2), J10.1 (Pin_1)
- net LED RED: now reaches J8.2 (Pin_2), R4.2
- net LED RED: now also J10.2 (Pin_2)
- net LED GREEN: now reaches J8.3 (Pin_3), R5.2
- net LED GREEN: now also J10.3 (Pin_3)
- net LED BLUE: now reaches J8.4 (Pin_4), R6.2
- net LED BLUE: now also J10.4 (Pin_4)
- net 3.3VDC: now reaches J4.3 (Pin_3), J7.1 (Pin_1)
- net 3.3VDC: now also J11.1 (Pin_1)
Other:
- moved on the sheet: J3, J4, J7, J8, J9, Q1, Q2, Q3, R1, R2, R3, R4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

Commit message: Added the kicad source file of the production batch
Parts:
- J7: value I2C BH1750 -> I2C BH1750 XH; footprint Connector_PinSocket_2.54mm:PinSocket_1x04_P2.54mm_Vertical -> Connector_JST:JST_XH_B4B-XH-AM_1x04_P2.50mm_Vertical
- J8: footprint Connector_PinSocket_2.54mm:PinSocket_1x04_P2.54mm_Vertical -> Connector_JST:JST_XH_B4B-XH-AM_1x04_P2.50mm_Vertical
